Commit message: use 7dof arm

File: caster_man_description/urdf/caster_man_xacro.xacro (robot description, xacro)
@@ -2,32 +2,27 @@
 <robot name = "caster_kinova_xacro" xmlns:xacro = "http://www.ros.org/wiki/xacro">
   <xacro:property name="M_PI" value="3.1415926535897931" />
-  <xacro:include filename="$(find kinova_description)/urdf/j2n6s300.xacro"/>
+  <!-- caster include -->
   <xacro:include filename = "$(find caster_description)/urdf/caster.urdf.xacro" />
+  <xacro:include filename = "$(find caster_body_description)/urdf/caster_body.urdf.xacro" />
+  <!-- sensor include -->
+  <xacro:include filename="$(find kinova_description)/urdf/j2s7s300.xacro" />
+  <xacro:include filename="$(find pan_tilt_description)/urdf/pan_tilt.urdf.xacro" />
+  <xacro:include filename="$(find caster_man_description)/urdf/kinect_v2.urdf.xacro" />
+  <!-- caster and caster_body -->
   <caster_robot/>
+  <xacro:caster_body parent="base_link">
+    <origin xyz="0.0 0.0 0.2755" rpy="0 0 0" />
+  </xacro:caster_body>
    <!-- realsense d435 -->
   <xacro:include filename="$(find caster_man_description)/urdf/realsense_d435.urdf.xacro" />
-  <link name="kinova_base">
-    <visual>
-        <origin xyz="0 0 0" rpy="0 0 0" />
-        <geometry>
-          <mesh filename="package://caster_man_description/mesh/kinova_base.STL" />
-        </geometry>
-        <material name="">
-          <color rgba="0.3 0.3 0.3 1.0" />
-        </material>
-      </visual>
-  </link>
-  <joint name="connect_caster_and_base" type="fixed">
-    <child link="kinova_base" />
-    <parent link="base_link" />
-    <origin xyz="-0.045 0 0.2745" rpy="0 0 0" />
+  <!-- kinova 7dof arm -->
+  <link name="arm_mount_link" />
+  <joint name="arm_mount_joint" type="fixed">
+    <origin xyz="0 0 0" rpy="${M_PI/2} 0 0" />
+    <parent link="caster_body_arm_link"/>
+    <child link="arm_mount_link"/>
   </joint>
-  <link name="kinova_mount_link" />
-  <joint name="kinova_mount" type="fixed">
-    <child link="kinova_mount_link" />
-    <parent link="kinova_base" />
-    <origin xyz="0 0 0.049" rpy="0 0 ${M_PI/2}" />
-  </joint>
-  <xacro:j2n6s300 base_parent="kinova_mount_link"/>
+  <xacro:j2s7s300 base_parent="arm_mount_link"/>
+  <!-- realsense -->
   <link name="realsense_coupling_link">
     <visual>
@@ -43,5 +38,5 @@
   <joint name="realsense_coupling_joint" type="fixed">
     <origin xyz="0 0 -0.015" rpy="${M_PI/2} ${M_PI/2} ${M_PI/2}" />
-    <parent link="j2n6s300_link_6"/>
+    <parent link="j2s7s300_link_7"/>
     <child link="realsense_coupling_link"/>
   </joint>
@@ -49,3 +44,11 @@
     <origin xyz="0.01005 0 0.0725" rpy="0 0 0"/>
   </sensor_d435>
+  <!-- pan tilt -->
+  <xacro:pan_tilt parent="caster_body_head_link" >
+    <origin xyz="0 0 0" rpy="0 0 0" />
+  </xacro:pan_tilt>
+  <!-- kinect -->
+  <xacro:kinect_v2 parent="pan_tilt_kinect_surface" >
+    <origin xyz="0 0 0" rpy="0 0 0" />
+  </xacro:kinect_v2>
 </robot>

Commit message: use new realsense coupling

File: caster_man_description/urdf/caster_man_xacro.xacro (robot description, xacro)
@@ -29,5 +29,5 @@
       <origin xyz="0 0 0" rpy="0 0 0" />
       <geometry>
-        <mesh filename="package://caster_man_description/mesh/ur3_realsense_coupling.stl" />
+        <mesh filename="package://caster_man_description/mesh/kinova_realsense_coupling.stl" />
       </geometry>
       <material name="">
@@ -37,10 +37,10 @@
   </link>
   <joint name="realsense_coupling_joint" type="fixed">
-    <origin xyz="0 0 -0.015" rpy="${M_PI/2} ${M_PI/2} ${M_PI/2}" />
+    <origin xyz="0 0 0.007" rpy="0 0 0" />
     <parent link="j2s7s300_link_7"/>
     <child link="realsense_coupling_link"/>
   </joint>
   <sensor_d435 parent="realsense_coupling_link" prefix="camera">
-    <origin xyz="0.01005 0 0.0725" rpy="0 0 0"/>
+    <origin xyz="0.0875 0 -0.01515" rpy="0 ${M_PI/2} 0"/>
   </sensor_d435>
   <!-- pan tilt -->

Commit message: use j2s6s200

File: caster_man_description/urdf/caster_man_xacro.xacro (robot description, xacro)
@@ -6,5 +6,5 @@
   <xacro:include filename = "$(find caster_description)/urdf/caster_body.urdf.xacro" />
   <!-- sensor include -->
-  <xacro:include filename="$(find kinova_description)/urdf/j2s7s300.xacro" />
+  <xacro:include filename="$(find kinova_description)/urdf/j2s6s200.xacro" />
   <xacro:include filename="$(find pan_tilt_description)/urdf/pan_tilt.urdf.xacro" />
   <xacro:include filename="$(find caster_man_description)/urdf/kinect_v2.urdf.xacro" />
@@ -12,9 +12,9 @@
   <caster_robot/>
   <xacro:caster_body parent="base_link">
-    <origin xyz="0.0 0.0 0.2755" rpy="0 0 0" />
+    <origin xyz="0.072 0.0 0.2815" rpy="0 0 0" />
   </xacro:caster_body>
    <!-- realsense d435 -->
   <xacro:include filename="$(find caster_man_description)/urdf/realsense_d435.urdf.xacro" />
-  <!-- kinova 7dof arm -->
+  <!-- kinova 6dof arm -->
   <link name="arm_mount_link" />
   <joint name="arm_mount_joint" type="fixed">
@@ -23,5 +23,5 @@
     <child link="arm_mount_link"/>
   </joint>
-  <xacro:j2s7s300 base_parent="arm_mount_link"/>
+  <xacro:j2s6s200 base_parent="arm_mount_link"/>
   <!-- realsense -->
   <link name="realsense_coupling_link">
@@ -38,5 +38,5 @@
   <joint name="realsense_coupling_joint" type="fixed">
     <origin xyz="0 0 0.007" rpy="0 0 0" />
-    <parent link="j2s7s300_link_7"/>
+    <parent link="j2s6s200_link_6"/>
     <child link="realsense_coupling_link"/>
   </joint>
@@ -46,5 +46,5 @@
   <!-- pan tilt -->
   <xacro:pan_tilt parent="caster_body_head_link" >
-    <origin xyz="0 0 0" rpy="0 0 0" />
+    <origin xyz="0 0 0.05" rpy="0 0 0" />
   </xacro:pan_tilt>
   <!-- kinect -->

Commit message: add j2s6s200 moveit

File: caster_man_description/urdf/caster_man_xacro.xacro (robot description, xacro)
@@ -8,5 +8,6 @@
   <xacro:include filename="$(find kinova_description)/urdf/j2s6s200.xacro" />
   <xacro:include filename="$(find pan_tilt_description)/urdf/pan_tilt.urdf.xacro" />
-  <xacro:include filename="$(find caster_man_description)/urdf/kinect_v2.urdf.xacro" />
+  <xacro:include filename="$(find pan_tilt_description)/urdf/kinect_v2.urdf.xacro" />
+  <xacro:include filename="$(find pan_tilt_description)/urdf/pan_tilt_neck_50mm.urdf.xacro" />
   <!-- caster and caster_body -->
   <caster_robot/>
@@ -45,6 +46,9 @@
   </sensor_d435>
   <!-- pan tilt -->
-  <xacro:pan_tilt parent="caster_body_head_link" >
-    <origin xyz="0 0 0.05" rpy="0 0 0" />
+  <xacro:pan_tilt_neck_50mm parent="caster_body_head_link" >
+    <origin xyz="0 0 0" rpy="0 0 0" />
+  </xacro:pan_tilt_neck_50mm>
+  <xacro:pan_tilt parent="pan_tilt_neck_top" >
+    <origin xyz="0 0 0" rpy="0 0 0" />
   </xacro:pan_tilt>
   <!-- kinect -->
